File: MWMWM.kicad_pcb (KiCad board)
At the start: 2 copper layers, 99.4 x 128.5 mm, 97 parts, among them J1 Conn_02x05_Odd_Even, J17 AudioJack2, J18 AudioJack2, J19 AudioJack2, J20 AudioJack2, Q1 BC857, Q2 BC847, U1 TL074, U2 TL074, U3 TL074, U4 LM13700

Commit message: Add files via upload
Parts:
- R15, R7: value 10k -> 47k
Changed lines of the file:
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@@
 			)
 		)
-		(property "Value" "10k"
+		(property "Value" "47k"
 			(at 0 -1.65 90)
 			(layer "B.Fab")
@@
 			)
 		)
-		(property "Value" "10k"
+		(property "Value" "47k"
 			(at 0 -1.65 90)
 			(layer "B.Fab")
@@
 	)
 	(gr_line
-		(start 21.807101 55.4)
-		(end 31.1964 66.874999)
-		(stroke
-			(width 0.1)
-			(type default)
-		)
-		(layer "F.SilkS")
-	)
-	(gr_line
-		(start 24.8 128.3)
-		(end 24.8107 112.9)
-		(stroke
-			(width 0.1)
-			(type default)
-		)
-		(layer "F.SilkS")
-	)
-	(gr_line
-		(start 24.8 128.3)
-		(end 31.33215 120.6)
-		(stroke
-			(width 0.1)
-			(type default)
-		)
-		(layer "F.SilkS")
-	)
-	(gr_line
-		(start 24.8107 112.9)
-		(end 21.807101 55.4)
-		(stroke
-			(width 0.1)
-			(type default)
-		)
-		(layer "F.SilkS")
-	)
-	(gr_line
-		(start 31.1964 44.074999)
-		(end 31.1964 66.874999)
-		(stroke
-			(width 0.1)
-			(type default)
-		)
-		(layer "F.SilkS")
-	)
-	(gr_line
-		(start 31.1964 66.874999)
-		(end 31.1964 89.674999)
-		(stroke
-			(width 0.1)
-			(type default)
-		)
-		(layer "F.SilkS")
-	)
-	(gr_line
-		(start 31.1964 89.674999)
-		(end 37.8107 112.9)
-		(stroke
-			(width 0.1)
-			(type default)
-		)
-		(layer "F.SilkS")
-	)
-	(gr_line
-		(start 37.8 128.3)
-		(end 37.8107 112.9)
-		(stroke
-			(width 0.1)
-			(type default)
-		)
-		(layer "F.SilkS")
-	)
-	(gr_line
